Commit message: mock(가짜 하드웨어)버전으로 ros2_contorl 테스트까지 완료.

File: src/my_omx_description/urdf/main.urdf.xacro (robot description, xacro)
@@ -15,3 +15,35 @@
     <child link="link1" />
   </joint>
+  <!-- ros2_control 설정 -->
+  <ros2_control name="MyOmxSystem" type="system">
+    <hardware>
+      <plugin>fake_components/GenericSystem</plugin>
+      <param name="mock_sensor_commands">false</param>
+    </hardware>
+    <joint name="joint1">
+      <command_interface name="position" />
+      <state_interface name="position" />
+      <state_interface name="velocity" />
+    </joint>
+    <joint name="joint2">
+      <command_interface name="position" />
+      <state_interface name="position" />
+      <state_interface name="velocity" />
+    </joint>
+    <joint name="joint3">
+      <command_interface name="position" />
+      <state_interface name="position" />
+      <state_interface name="velocity" />
+    </joint>
+    <joint name="joint4">
+      <command_interface name="position" />
+      <state_interface name="position" />
+      <state_interface name="velocity" />
+    </joint>
+    <joint name="gripper_left_joint">
+      <command_interface name="position" />
+      <state_interface name="position" />
+      <state_interface name="velocity" />
+    </joint>
+  </ros2_control>
 </robot>

Commit message: 분기버전으로 mock 버전 완료. 코드 분석 필요함.

File: src/my_omx_description/urdf/main.urdf.xacro (robot description, xacro)
@@ -2,12 +2,27 @@
 <!-- OpenManipulator Chain -->
 <robot name="open_manipulator_x" xmlns:xacro="http://ros.org/wiki/xacro">
-  <!-- Import URDF -->
-  <xacro:include
-    filename="$(find my_omx_description)/urdf/manipulator.urdf.xacro" />
-  <!-- Instantiate the macro -->
+  <!-- 런치 인자 선언 -->
+  <xacro:arg name="use_fake_hardware" default="true" />
+  <!-- ============================= -->
+  <!-- Include 필요한 xacro -->
+  <!-- ============================= -->
+  <xacro:include filename="$(find my_omx_description)/urdf/manipulator.urdf.xacro" />
+  <xacro:include filename="$(find my_omx_description)/ros2_control/my_omx_system.ros2_control.xacro" />
+  <!-- ============================= -->
+  <!-- 매크로 호출 (모델 + ros2_control) -->
+  <!-- ============================= -->
+  <!-- 로봇 링크/조인트 정의 -->
   <xacro:open_manipulator_x prefix="" />
-  <!-- World -->
+  <!-- ros2_control 시스템 연결 -->
+  <xacro:my_omx_system
+    name="MyOmxSystem"
+    prefix=""
+    port_name="/dev/ttyUSB0"
+    use_fake_hardware="$(arg use_fake_hardware)"
+  />
+  <!-- ============================= -->
+  <!-- World 프레임 고정 -->
+  <!-- ============================= -->
   <link name="world" />
-  <!-- World fixed joint-->
   <joint name="world_fixed" type="fixed">
     <origin xyz="0 0 0" rpy="0 0 0" />
@@ -15,35 +30,3 @@
     <child link="link1" />
   </joint>
-  <!-- ros2_control 설정 -->
-  <ros2_control name="MyOmxSystem" type="system">
-    <hardware>
-      <plugin>fake_components/GenericSystem</plugin>
-      <param name="mock_sensor_commands">false</param>
-    </hardware>
-    <joint name="joint1">
-      <command_interface name="position" />
-      <state_interface name="position" />
-      <state_interface name="velocity" />
-    </joint>
-    <joint name="joint2">
-      <command_interface name="position" />
-      <state_interface name="position" />
-      <state_interface name="velocity" />
-    </joint>
-    <joint name="joint3">
-      <command_interface name="position" />
-      <state_interface name="position" />
-      <state_interface name="velocity" />
-    </joint>
-    <joint name="joint4">
-      <command_interface name="position" />
-      <state_interface name="position" />
-      <state_interface name="velocity" />
-    </joint>
-    <joint name="gripper_left_joint">
-      <command_interface name="position" />
-      <state_interface name="position" />
-      <state_interface name="velocity" />
-    </joint>
-  </ros2_control>
 </robot>
